File: Hardware/DumbDrehscheibenDecoder/DumbDrehscheibenDecoder.kicad_pcb (KiCad board)
At the start: 2 copper layers, 50 x 50 mm, 13 parts, among them J1 Screw_Terminal_01x03, J2 Screw_Terminal_01x04, K1 HFD2, K2 HFD2-L2, U1 ULN2003A

Commit message: Updated the PCB
Parts:
- removed K1: HFD2, RelayDeltaphi:HFD
- removed K2: HFD2-L2, RelayDeltaphi:HFD2-L2
- added D3: 1N4001, Diode_THT:D_A-405_P7.62mm_Horizontal, F.Cu at (26.7, 64.8)
- added R1: 22k, Resistor_THT:R_Axial_DIN0204_L3.6mm_D1.6mm_P7.62mm_Horizontal, F.Cu at (22.9, 64.8)
- added R2: 220, Resistor_THT:R_Axial_DIN0204_L3.6mm_D1.6mm_P7.62mm_Horizontal, F.Cu at (27.3, 52.1)
- added R3: 22k, Resistor_THT:R_Axial_DIN0204_L3.6mm_D1.6mm_P7.62mm_Horizontal, F.Cu at (8.26, 41.3)
- added SW1: SW_Push, Button_Switch_THT:SW_PUSH_6mm, F.Cu at (10.8, 45.7)
- added U2: LTV-817, Package_DIP:DIP-4_W7.62mm, F.Cu at (24.1, 62.2)
- J1: value Screw_Terminal_01x03 -> Screw_Terminal_01x04; footprint TerminalBlock_RND:TerminalBlock_RND_205-00002_1x03_P5.00mm_Horizontal -> TerminalBlock_RND:TerminalBlock_RND_205-00003_1x04_P5.00mm_Horizontal
- U1: value ULN2003A -> L293D; footprint Package_DIP:DIP-16_W7.62mm_Socket -> Package_DIP:DIP-16_W7.62mm; moved to F.Cu
- moved H1 31.9 mm to (23.5, 36.2)
- moved H3 21.0 mm to (66.7, 36.2)
- moved U1 19.0 mm to (50.8, 48.3), turned to 0 degrees
- moved H2 17.3 mm to (23.5, 79.4)
- moved D1 12.2 mm to (52.7, 73.7)
- moved D2 11.4 mm to (52.7, 69.8)
- moved J1 11.4 mm to (66.0, 58.4)
- moved J2 8.91 mm to (31.8, 79.4)
- moved A1 7.62 mm to (45.7, 69.8)
- moved C1 6.98 mm to (54.0, 41.9)
- moved H4 0.90 mm to (66.7, 79.4)
Connections:
- net Net-(A1-Pad30) renamed /MM_Vin
- net Net-(D1-Pad3) renamed /MM_B
- net Net-(D1-Pad4) renamed /MM_0
- net Net-(D2-Pad3) renamed /PWR_B
- net Net-(D2-Pad4) renamed /PWR_0
- A1 pad 12: (no net) -> Net-(A1-Pad12)
- A1 pad 19: (no net) -> Net-(A1-Pad19)
- A1 pad 5: (no net) -> /MM_Sense
- A1 pad 6: (no net) -> Net-(A1-Pad6)
- A1 pad 7: (no net) -> Net-(A1-Pad7)
- D2 pad 1: Net-(D2-Pad1) -> /Pwr_Vin
- D2 pad 2: Net-(D2-Pad2) -> GND
- J1 pad 1: Net-(J1-Pad1) -> /MOT_3Y
- J1 pad 2: Net-(J1-Pad2) -> /MOT_4Y
- J1 pad 3: Net-(J1-Pad3) -> /MOT_2Y
- U1 pad 1: (no net) -> Net-(A1-Pad9)
- U1 pad 10: (no net) -> Net-(A1-Pad8)
- U1 pad 11: Net-(K1-Pad16) -> /MOT_3Y
- U1 pad 12: Net-(K2-Pad15) -> GND
- U1 pad 13: Net-(K2-Pad16) -> GND
- U1 pad 14: (no net) -> /MOT_4Y
- U1 pad 15: (no net) -> Net-(A1-Pad10)
- U1 pad 16: (no net) -> VCC
- U1 pad 2: (no net) -> Net-(A1-Pad12)
- U1 pad 3: (no net) -> /MOT_1Y
- U1 pad 4: (no net) -> GND
- U1 pad 5: Net-(A1-Pad10) -> GND
- U1 pad 6: Net-(A1-Pad9) -> /MOT_2Y
- U1 pad 7: Net-(A1-Pad8) -> Net-(A1-Pad7)
- U1 pad 8: GND -> /Pwr_Vin
- U1 pad 9: GND -> Net-(A1-Pad6)
Routing:
- net VCC: track 83.0 -> 8.19 mm
- net /MM_0: track 0.00 -> 57.5 mm
- net /MM_B: track 0.00 -> 47.0 mm
- net Net-(J1-Pad3): track 37.1 -> 0.00 mm
- net Net-(K2-Pad16): track 30.7 -> 0.00 mm
- net Net-(K2-Pad15): track 29.6 -> 0.00 mm
- net Net-(D2-Pad1): track 29.6 -> 0.00 mm
- net /MOT_2Y: track 0.00 -> 27.7 mm
- net /MM_Sense: track 0.00 -> 26.4 mm
- net Net-(D2-Pad2): track 26.2 -> 0.00 mm
- net /MM_Vin: track 0.00 -> 23.8 mm
- net Net-(J1-Pad2): track 22.2 -> 0.00 mm
- net /MOT_1Y: track 0.00 -> 21.6 mm
- net Net-(A1-Pad8): track 2.54 -> 21.3 mm
- net Net-(A1-Pad6): track 0.00 -> 18.1 mm
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- added copper zone on B.Cu, net GND
- added copper zone on F.Cu, net GND
