File: Hardware/DumbDrehscheibenDecoder/DumbDrehscheibenDecoder.sch (KiCad schematic (older format))
At the start: 13 parts, among them J1 Screw_Terminal_01x03, J2 Screw_Terminal_01x04, K1 HFD2, K2 HFD2-L2, U1 ULN2003A

Commit message: Updated the PCB
Parts:
- removed J1: Screw_Terminal_01x03, TerminalBlock_RND:TerminalBlock_RND_205-00002_1x03_P5.00mm_Horizontal, symbol Connector:Screw_Terminal_01x03
- removed K1: HFD2, RelayDeltaphi:HFD, symbol RelayDeltaphi:HFD2
- removed K2: HFD2-L2, RelayDeltaphi:HFD2-L2, symbol RelayDeltaphi:HFD2-L2
- removed U1: ULN2003A, Package_DIP:DIP-16_W7.62mm_Socket, symbol Transistor_Array:ULN2003A
- added D3: 1N4001, Diode_THT:D_A-405_P7.62mm_Horizontal, symbol Device:D
- added J1: Screw_Terminal_01x04, TerminalBlock_RND:TerminalBlock_RND_205-00003_1x04_P5.00mm_Horizontal, symbol Connector:Screw_Terminal_01x04
- added R1, R3: 22k, Resistor_THT:R_Axial_DIN0204_L3.6mm_D1.6mm_P7.62mm_Horizontal, symbol Device:R
- added R2: 220, Resistor_THT:R_Axial_DIN0204_L3.6mm_D1.6mm_P7.62mm_Horizontal, symbol Device:R
- added SW1: SW_Push, Button_Switch_THT:SW_PUSH_6mm, symbol Switch:SW_Push
- added U1: L293D, Package_DIP:DIP-16_W7.62mm, symbol Driver_Motor:L293D
- added U2: LTV-817, Package_DIP:DIP-4_W7.62mm, symbol Isolator:LTV-817
Connections:
- net labels added: MM_0, MM_B, MM_Sense, MM_Vin, MOT_1Y, MOT_2Y, MOT_3Y, MOT_4Y, PWR_0, PWR_B, Pwr_Vin
- wire segments 83 -> 91
